File: hardware/kicad8.0/light_rail.kicad_pcb (KiCad board)
At the start: 4 copper layers, 73.4 x 100.5 mm, 211 parts, among them J1 USB_C_Receptacle_USB2.0_16P, J2 Conn_01x04_Pin, J3 AVR-ISP-6, SW1 SW_Push, SW10 SW_Push, SW11 SW_Push, SW12 SW_Push, SW13 SW_Push, SW14 SW_SPST, SW2 SW_Push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

Commit message: changes for fab
Parts:
- moved C4 0.36 mm to (34.4, 82.1)
- moved U3 0.23 mm to (68.3, 40.0)
Routing:
- net SEGA: track 31.4 -> 29.3 mm
- net SEGG: track 41.3 -> 39.5 mm
- net SEGC: track 34.6 -> 33.2 mm
- net SEGB: track 32.4 -> 31.1 mm
- net +3V3: track 103.5 -> 104.7 mm
- net SEGF: track 34.9 -> 34.0 mm
- net CB5: track 122.0 -> 122.6 mm
- net SEGD: track 32.7 -> 33.2 mm
- net GND: track 224.5 -> 224.0 mm
Other:
- outline, holes or cut-outs redrawn
- board text added: "WayWayWay"

Commit message: fab updates 2
Parts:
- removed the G*** at (50.9, 72.8)
- added G***: LOGO, Light_Rail:TrainDrawing, B.Cu at (51.7, 76.5)
- added H1: MountingHole, Light_Rail:MountingHole_Custom, F.Cu at (19.1, 26.3)
- added H2: MountingHole, Light_Rail:MountingHole_Custom, F.Cu at (83.3, 26.3)
- added H3: MountingHole, Light_Rail:MountingHole_Custom, F.Cu at (19.1, 117.6)
- added H4: MountingHole, Light_Rail:MountingHole_Custom, F.Cu at (83.3, 117.6)
- moved G*** 3.98 mm to (73.5, 52.4)
- moved J3 3.49 mm to (27.3, 120.4)
- moved J2 1.62 mm to (68.6, 120.4)
- renumbered C2 to C1, C1 to C2
Routing:
- net GND: track 224.0 -> 236.8 mm, vias 23 -> 20
- net RST: track 58.9 -> 55.2 mm
- net SDA: track 125.0 -> 127.4 mm
- net +3V3: track 104.7 -> 102.4 mm, vias 16 -> 14
- net SEGDP: track 30.9 -> 28.7 mm
- net MOSI: track 44.7 -> 46.4 mm
- net SCK: track 49.3 -> 51.0 mm
- net SCL: track 132.8 -> 134.4 mm
- net MISO: track 51.3 -> 52.6 mm
- net CA7: track 164.7 -> 165.8 mm
- net Net-(U1-XTAL1): track 6.27 -> 5.31 mm
- net CA9: track 119.7 -> 119.1 mm
Other:
- outline, holes or cut-outs redrawn
